File: pcb/teensy/user_interface_teensy.sch (KiCad schematic (older format))
At the start: 15 parts, among them P1 HEADER_02X08_SMD, SW1 SPST_SLIDE_AS, U1 TLE7230R

Commit message: Progress towards schematic v1.0.
Parts:
- removed C1: 10uF, user_interface_teensy:SM1210, symbol 10uF
- removed C2: 0.1uF, user_interface_teensy:SM1210, symbol 0.1uF
- removed L1, L2, L3, L4, L5, L6, L7, L8, L9: LED_24V, user_interface_teensy:LED_555-3XXX, symbol LED_24V
- removed P1: HEADER_02X08_SMD, user_interface_teensy:HEADER_02x08_SMD, symbol HEADER_02X08_SMD
- removed SW1: SPST_SLIDE_AS, user_interface_teensy:SPST_SLIDE_AS, symbol SPST_SLIDE_AS
- removed U1: TLE7230R, user_interface_teensy:PG-DSO-36, symbol TLE7230R
- added C?: 10uF, footprints:SM1210, symbol 10uF
- added NHD?: NHD-ASC3-169, footprints:NHD-ASC3, symbol NHD-ASC3-169
Connections:
- net labels added: CD, OLEDCS, OLEDDC, SDCS
- net labels removed: CS, LED_PWR, OUT0, OUT1, OUT2, OUT3, OUT4, OUT5, OUT6, OUT7
- wire segments 85 -> 28
- no-connect marks 25 -> 24

Commit message: Progress towards teensy v1.0.
Parts:
- added C2: 10uF_2917_POL, user_interface_teensy:SM2917_POL, symbol 10uF_2917_POL
- added C3, C4, C5, C6, C7, C8: 0.1uF, user_interface_teensy:SM1210, symbol 0.1uF
- added E1: ENCODER_62A11-02-P, user_interface_teensy:ENCODER_62AVD, symbol ENCODER_62A11-02-P
- added J1: JOYSTICK, user_interface_teensy:JOYSTICK, symbol JOYSTICK
- added SW1, SW2, SW3: KT_SWITCH, user_interface_teensy:KT_SWITCH, symbol KT_SWITCH
- added U1, U2, U3, U4: MAX6817, user_interface_teensy:MAX6817, symbol MAX6817
- C1: renamed from C?; footprint footprints:SM1210 -> user_interface_teensy:SM1210
- MDT1: footprint user_interface_teensy:MODULAR_DEVICE_TEENSY -> user_interface_teensy:MODULAR_DEVICE_TEENSY_MALE
- NHD1: renamed from NHD?; footprint footprints:NHD-ASC3 -> user_interface_teensy:NHD-ASC3
Connections:
- net CD: now also MDT1.14 (D14/A0/SCKB)
- net GND: now also C2.2, C3.2, C4.2, C5.2, C6.2, C7.2, C8.2, E1.1 (GND), E1.2 (BTN_B), J1.COM, SW1.3, SW2.3, SW3.3, U1.2 (GND), U2.2 (GND), U3.2 (GND), U4.2 (GND)
- net OLEDDC: now also MDT1.29 (D29/A18/SCL1)
- net SDCS: now also MDT1.9 (D9/RX2/PWM/ICP/CSB/I2SBCLK)
- net VEE: now also C2.1, C3.1, C4.1, C5.1, C6.1, C7.1, C8.1, E1.6 (+5VDC), U1.5 (Vcc), U2.5 (Vcc), U3.5 (Vcc), U4.5 (Vcc)
- net BTN_ENC: now reaches MDT1.15 (D15/A1/TOUCH/CSB)
- net BTN_ENC: now also U1.6 (OUT1)
- net BTN_CALL: now reaches MDT1.16 (D16/A2/TOUCH)
- net BTN_CALL: now also U1.4 (OUT2)
- net LEFT: now reaches MDT1.17 (D17/A3/TOUCH)
- net LEFT: now also U2.6 (OUT1)
- net RIGHT: now reaches MDT1.18 (D18/A4/SDA0/TOUCH)
- net RIGHT: now also U2.4 (OUT2)
- net UP: now reaches MDT1.19 (D19/A5/SCL0/TOUCH)
- net UP: now also U3.6 (OUT1)
- net DOWN: now reaches MDT1.20 (D20/A6/PWM/CSB)
- net DOWN: now also U3.4 (OUT2)
- net BTN_A: now reaches MDT1.21 (D21/A7/PWM/RX1B/CSB)
- net BTN_A: now also U4.6 (OUT1)
- net BTN_B: now reaches MDT1.22 (D22/A8/TOUCH/PWM/ICP/I2STX)
- net BTN_B: now also U4.4 (OUT2)
- net ENC_B: now reaches MDT1.4 (D4/PWM/CANRX)
- net ENC_B: now also E1.4 (OUT_B)
- net PWM renamed ENC_A
- net ENC_A: now also E1.5 (OUT_A)
- net VDD: no longer names the net of MDT1.VDD (VDD_(+9-42VDC))
- new net B_BTN_A: SW2.2, U4.1 (IN1)
- new net B_BTN_B: SW3.2, U4.3 (IN2)
- new net B_BTN_CALL: SW1.2, U1.3 (IN2)
- new net B_BTN_ENC: E1.3 (BTN_A), U1.1 (IN1)
- new net B_DOWN: J1.D (DOWN), U3.3 (IN2)
- new net B_LEFT: J1.L (LEFT), U2.1 (IN1)
- new net B_RIGHT: J1.R (RIGHT), U2.3 (IN2)
- new net B_UP: J1.U (UP), U3.1 (IN1)
- no-connect marks 24 -> 13
Other:
- moved on the sheet: NHD1

Commit message: Finished pcb v1.0.
Parts:
- added S1: HEADER_01X02_SHR, user_interface_teensy:Header_Shrouded_2_Pin, symbol HEADER_01X02_SHR
Connections:
- net labels removed: CD
- wire segments 101 -> 102
- no-connect marks 13 -> 15
Changed lines of the file:
@@
 LIBS:components
 LIBS:user_interface_teensy
-LIBS:user_interface_teensy-cache
 EELAYER 25 0
 EELAYER END
@@
 Wire Wire Line
 	6400 1800 6100 1800
-Wire Wire Line
-	6400 2000 6100 2000
 $Comp
 L VEE #PWR05
@@
 Text Label 6100 1800 0    60   ~ 0
 SDCS
-Text Label 6100 2000 0    60   ~ 0
-CD
 NoConn ~ 7400 1100
 $Comp
@@
 OLEDDC
 Wire Wire Line
-	3850 2150 3950 2150
-Text Label 3950 2150 0    60   ~ 0
-CD
-Wire Wire Line
 	3850 2050 3950 2050
 Wire Wire Line
@@
 Wire Wire Line
 	3850 1450 3950 1450
-Wire Wire Line
-	3850 1350 3950 1350
 Text Label 3950 2050 0    60   ~ 0
 BTN_ENC
-Text Label 3950 1950 0    60   ~ 0
+Text Label 3950 2150 0    60   ~ 0
 BTN_CALL
 Text Label 3950 1850 0    60   ~ 0
 LEFT
-Text Label 3950 1750 0    60   ~ 0
+Text Label 3950 1950 0    60   ~ 0
 RIGHT
 Text Label 3950 1650 0    60   ~ 0
 UP
-Text Label 3950 1550 0    60   ~ 0
+Text Label 3950 1750 0    60   ~ 0
 DOWN
 Text Label 3950 1450 0    60   ~ 0
 BTN_A
-Text Label 3950 1350 0    60   ~ 0
+Text Label 3950 1550 0    60   ~ 0
 BTN_B
 Wire Wire Line
@@
 Text Label 1050 1450 0    60   ~ 0
 ENC_B
+NoConn ~ 6400 2000
+Wire Wire Line
+	3850 2150 3950 2150
+NoConn ~ 3850 1350
+$Comp
+L HEADER_01X02_SHR S1
+U 1 1 57C083F3
+P 7900 4700
+F 0 "S1" H 7900 4850 50  0000 C CNN
+F 1 "HEADER_01X02_SHR" V 8000 4700 50  0000 C CNN
+F 2 "user_interface_teensy:Header_Shrouded_2_Pin" H 7800 4750 60  0001 C CNN
+F 3 "" H 7900 4700 60  0000 C CNN
+F 4 "digikey" H 8000 4950 60  0001 C CNN "Vendor"
+F 5 "WM4800-ND" H 8100 5050 60  0001 C CNN "PartNumber"
+F 6 "CONN HEADER 2POS .100 VERT GOLD" H 8200 5150 60  0001 C CNN "Description"
+	1    7900 4700
+	1    0    0    -1
+$EndComp
+$Comp
+L GND #PWR036
+U 1 1 57C086A8
+P 7650 4800
+F 0 "#PWR036" H 7650 4550 50  0001 C CNN
+F 1 "GND" H 7655 4627 50  0000 C CNN
+F 2 "" H 7650 4800 50  0000 C CNN
+F 3 "" H 7650 4800 50  0000 C CNN
+	1    7650 4800
+	1    0    0    -1
+$EndComp
+Wire Wire Line
+	7650 4800 7650 4750
+Wire Wire Line
+	7650 4750 7700 4750
+Wire Wire Line
+	7700 4650 7150 4650
+Text Label 7150 4650 0    60   ~ 0
+B_BTN_CALL
 $EndSCHEMATC
